File: Hardware/SCS Interface V1/KiCad/SCS_Interface.kicad_sch (KiCad schematic)
At the start: 37 parts, among them J1 SCS, J2 Headder, Q1 MMBTA06, Q2 MMBTA06, U1 LMR51420, U2 AZ1117CH2 - 3.3

Commit message: Update PCB after first pcb build
- Replace input detection
Parts:
- removed D2, D3: BAS31, Package_TO_SOT_SMD:SOT-23, symbol Device:D_Dual_Series_AKC_Parallel
- removed D5: M2, Diode_SMD:D_SMA, symbol Diode:1N4001
- removed Q2: MMBTA06, Package_TO_SOT_SMD:SOT-23, symbol Transistor_BJT:2SC4213
- added D2: ABS2, Diode_SMD:Diode_Bridge_Diotec_ABS, symbol Diode_Bridge:ABS2
- added D3: FDLL4148, Diode_SMD:D_MiniMELF, symbol Diode:1N4001
- added R10, R9: 10k, Resistor_SMD:R_0805_2012Metric, symbol Device:R
- added U3: LM397, Package_TO_SOT_SMD:SOT-23-5, symbol Comparator:LM397
- C5: value 1n -> 13p (OPT)
- D1: value TPSMC33A -> P4SMA39CA; footprint Diode_SMD:D_SMC -> Diode_SMD:D_SMA
- J1: footprint TerminalBlock_Phoenix:TerminalBlock_Phoenix_MKDS-1,5-2_1x02_P5.00mm_Horizontal -> TerminalBlock_Phoenix:TerminalBlock_Phoenix_MKDS-1,5-2_1x02_P5.00mm_Horizontal_PNP
- R4: value 100k -> 10k; Ref constructeurs CR0805-FX-1003ELF -> CR0805-FX-1002ELF
- R5: Ref constructeurs CR0805-FX-1002ELF -> CR0805-FX-1003ELF
- R6: value 10k -> 20k
Connections:
- net +3V3: now also R4.2, R6.2, U3.5 (V+); no longer R5.2
- net GND: now also D2.2 (-), D3.2 (A), R9.1, U3.2 (V-)
- net SCS_BUS_CC: now also D2.1 (+)
- net SCS_OUT: now also R10.1, U3.4; no longer C5.2, R6.1
- net VCC_IO: now also R10.2; no longer R6.2
- net at C1.1, D1.2 (A2), F1.2: now also D2.3
- net at C2.2, D1.1 (A1), L2.2: now also D2.4
- new net: R6.1, R9.2, U3.3 (+)
- new net: C5.2, D3.1 (K), R5.2, U3.1 (-)
Other:
- moved on the sheet: C6, Q1, R1, R2
